Commit message: Bug Fix

File: description/gazebo_control.xacro (robot description, xacro)
@@ -2,9 +2,9 @@
 <robot xmlns:xacro="http://www.ros.org/wiki/xacro">
     <gazebo>
-        <plugin name="diff_drive" filename="libgazeboros_diff_drive.so">
+        <plugin name="diff_drive" filename="libgazebo_ros_diff_drive.so">
             <!-- Wheel Information -->
             <left_joint>left_wheel_joint</left_joint>
             <right_joint>right_wheel_joint</right_joint>
-            <wheel_seperation>0.1905</wheel_seperation>
+            <wheel_separation>0.1905</wheel_separation>
             <wheel_diameter>0.065</wheel_diameter>
             <!-- Limits -->

File: description/robot.urdf.xacro (robot description, xacro)
@@ -1,5 +1,5 @@
 <?xml version="1.0"?>
 <robot xmlns:xacro="http://www.ros.org/wiki/xacro"  name="robot">
+    <xacro:include filename="gazebo_control.xacro"/>
     <xacro:include filename="robot_core.xacro"/>
-    <xacro:include filename="gazebo_control.xacro"/>
 </robot>

File: description/robot_core.xacro (robot description, xacro)
@@ -25,5 +25,5 @@
     <link name="chassis">
         <visual>
-            <origin xyz="0.175 0 0.0225"/>
+            <origin xyz="0.175 0 0.0275"/>
             <geometry>
                 <box size ="0.35 0.155 0.055"/>
@@ -32,5 +32,5 @@
         </visual>
         <collision>
-            <origin xyz="0.175 0 0.0225"/>
+            <origin xyz="0.175 0 0.0275"/>
             <geometry>
                 <box size ="0.35 0.155 0.055"/>
@@ -38,5 +38,5 @@
         </collision>
         <xacro:inertial_box mass="0.5" x="0.35" y="0.155" z="0.055">
-            <origin xyz="0.175 0 0.0225" rpy="0 0 0"/>
+            <origin xyz="0.175 0 0.0275" rpy="0 0 0"/>
         </xacro:inertial_box>
     </link>
@@ -69,5 +69,5 @@
     </link>
     <gazebo reference="left_wheel">
-        <material>Gazebo/Blue</material>
+        <material>Gazebo/Red</material>
     </gazebo>
     <!-- RIGHT WHEEL LINK -->
@@ -96,5 +96,5 @@
     </link>
     <gazebo reference="right_wheel">
-        <material>Gazebo/Blue</material>
+        <material>Gazebo/Red</material>
     </gazebo>
     <!-- CASTER WHEEL LINK -->
