Commit message: Camera Launch

File: description/lidar.xacro (robot description, xacro)
@@ -27,5 +27,5 @@
     <sensor name ="laser" type="ray">
         <pose>0 0 0 0 0 0</pose>
-        <visualize>true</visualize>
+        <visualize>false</visualize>
         <update_rate>10</update_rate>
         <ray>

File: description/robot.urdf.xacro (robot description, xacro)
@@ -4,3 +4,4 @@
     <xacro:include filename="robot_core.xacro"/>
     <xacro:include filename="lidar.xacro"/>
+    <xacro:include filename="camera.xacro"/>
 </robot>

File: description/robot_core.xacro (robot description, xacro)
@@ -72,5 +72,5 @@
     </link>
     <gazebo reference="left_wheel">
-        <material>Gazebo/Red</material>
+        <material>Gazebo/Blue</material>
     </gazebo>
     <!-- RIGHT WHEEL LINK -->
@@ -99,5 +99,5 @@
     </link>
     <gazebo reference="right_wheel">
-        <material>Gazebo/Red</material>
+        <material>Gazebo/Blue</material>
     </gazebo>
     <!-- CASTER WHEEL LINK -->
