Commit message: RPLidar Launch

File: description/robot.urdf.xacro (robot description, xacro)
@@ -3,3 +3,4 @@
     <xacro:include filename="gazebo_control.xacro"/>
     <xacro:include filename="robot_core.xacro"/>
+    <xacro:include filename="lidar.xacro"/>
 </robot>

File: description/robot_core.xacro (robot description, xacro)
@@ -13,4 +13,7 @@
     <material name="black">
         <color rgba="0 0 0 1" />
+    </material>
+    <material name="red">
+        <color rgba="1 0 0 1" />
     </material>
     <!-- BASE LINK -->

Commit message: setup ros2_control

File: description/robot.urdf.xacro (robot description, xacro)
@@ -1,5 +1,11 @@
 <?xml version="1.0"?>
 <robot xmlns:xacro="http://www.ros.org/wiki/xacro"  name="robot">
+    <xacro:arg name="use_ros2_control" default="true"/>
+    <xacro:if value="$(arg use_ros2_control)">
+    <xacro:include filename="ros2_control.xacro"/>
+    </xacro:if>
+    <xacro:unless value="$(arg use_ros2_control)">
     <xacro:include filename="gazebo_control.xacro"/>
+   </xacro:unless>
     <xacro:include filename="robot_core.xacro"/>
     <xacro:include filename="lidar.xacro"/>

File: description/robot_core.xacro (robot description, xacro)
@@ -63,5 +63,5 @@
         <collision>
             <geometry>
-                <cylinder radius="0.0325" length="0.04"/>
+                <sphere radius="0.0325"/>
             </geometry>
             <material name="blue"/>
@@ -90,5 +90,5 @@
         <collision>
             <geometry>
-                <cylinder radius="0.0325" length="0.04"/>
+                <sphere radius="0.0325"/>
             </geometry>
             <material name="blue"/>
